Commit message: Add tiago

File: tiago/tiago_mujoco/model/tiago.urdf (robot description, URDF)
Before this commit: robot tiago, 89 links, 88 joints
Links:
- link arm_1_link: geometry collision mesh filename=package://tiago_description/meshes/arm/arm_1.stl scale=1 1 1; visual mesh filename=package://tiago_description/meshes/arm/arm_1_visual.dae scale=1 1 1
- link arm_2_link: geometry collision mesh filename=package://tiago_description/meshes/arm/arm_2.stl scale=1 1 1; visual mesh filename=package://tiago_description/meshes/arm/arm_2_visual.dae scale=1 1 1
- link arm_3_link: geometry collision mesh filename=package://tiago_description/meshes/arm/arm_3.stl scale=1 1 1; visual mesh filename=package://tiago_description/meshes/arm/arm_3_visual.dae scale=1 1 1
- link arm_4_link: geometry collision mesh filename=package://tiago_description/meshes/arm/arm_4.stl scale=1 1 1; visual mesh filename=package://tiago_description/meshes/arm/arm_4_visual.dae scale=1 1 1
- link arm_5_link: geometry collision mesh filename=package://tiago_description/meshes/arm/arm_5-wrist-2010.stl scale=1 1 1; visual mesh filename=package://tiago_description/meshes/arm/arm_5_visual-wrist-2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 scale=1 1 1
- link arm_6_link: geometry collision mesh filename=package://tiago_description/meshes/arm/arm_6-wrist-2010.stl scale=1 1 1; visual mesh filename=package://tiago_description/meshes/arm/arm_6_visual-wrist-2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 scale=1 1 1
- link base_antenna_left_link: geometry collision mesh filename=package://pmb2_description/meshes/objects/antenna.stl; visual cylinder length=0.17 radius=0.005
- link base_antenna_right_link: geometry collision mesh filename=package://pmb2_description/meshes/objects/antenna.stl; visual cylinder length=0.17 radius=0.005
- link base_cover_link: geometry collision mesh filename=package://pmb2_description/meshes/base/base_ring.stl
- link base_laser_link: geometry collision mesh filename=package://pmb2_description/meshes/sensors/sick_tim551.stl
- link base_link: geometry collision mesh filename=package://pmb2_description/meshes/base/base.stl; visual mesh filename=package://pmb2_description/meshes/base/base_collision.stl
- link base_sonar_01_link: geometry collision mesh filename=package://pmb2_description/meshes/sensors/srf05.stl
- link base_sonar_02_link: geometry collision mesh filename=package://pmb2_description/meshes/sensors/srf05.stl
- link base_sonar_03_link: geometry collision mesh filename=package://pmb2_description/meshes/sensors/srf05.stl
- link caster_back_left_1_link: geometry collision mesh filename=package://pmb2_description/meshes/wheels/caster_1.stl
- link caster_back_left_2_link: geometry collision mesh filename=package://pmb2_description/meshes/wheels/caster_2.stl; visual sphere radius=0.025
- link caster_back_right_1_link: geometry collision mesh filename=package://pmb2_description/meshes/wheels/caster_1.stl
- link caster_back_right_2_link: geometry collision mesh filename=package://pmb2_description/meshes/wheels/caster_2.stl; visual sphere radius=0.025
- link caster_front_left_1_link: geometry collision mesh filename=package://pmb2_description/meshes/wheels/caster_1.stl
- link caster_front_left_2_link: geometry collision mesh filename=package://pmb2_description/meshes/wheels/caster_2.stl; visual sphere radius=0.025
- link caster_front_right_1_link: geometry collision mesh filename=package://pmb2_description/meshes/wheels/caster_1.stl
- link caster_front_right_2_link: geometry collision mesh filename=package://pmb2_description/meshes/wheels/caster_2.stl; visual sphere radius=0.025
- link hand_palm_link: geometry collision mesh filename=package://hey5_description/meshes/palm.stl scale=1 1 1; visual mesh filename=package://hey5_description/meshes/palm_collision.stl scale=1 1 1
- link hand_safety_box: geometry visual box size=0.2 0.115 0.18
- link head_1_link: geometry collision mesh filename=package://tiago_description/meshes/head/head_1.stl scale=1 1 1; visual mesh filename=package://tiago_description/meshes/head/head_1_visual.dae scale=1 1 1
- link head_2_link: geometry collision mesh filename=package://tiago_description/meshes/head/head_2.stl scale=1 1 1; visual mesh filename=package://tiago_description/meshes/head/head_2_visual.dae scale=1 1 1
- link torso_fixed_column_link: geometry collision box size=0.18 0.2 0.55; visual box size=0.23 0.23 0.55
- link torso_fixed_link: geometry collision mesh filename=package://tiago_description/meshes/torso/torso_fix.stl scale=1 1 1; visual box size=0.25 0.25 0.1
- link torso_lift_link: geometry collision mesh filename=package://tiago_description/meshes/torso/torso_lift_with_ar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 scale=1 1 1; visual mesh filename=package://tiago_description/meshes/torso/torso_lift_visual_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 scale=1 1 1
- link wheel_left_link: geometry collision mesh filename=package://pmb2_description/meshes/wheels/wheel.stl; visual sphere radius=0.0985
- link wheel_right_link: geometry collision mesh filename=package://pmb2_description/meshes/wheels/wheel.stl; visual sphere radius=0.0985

Commit message: Fix urdf

File: tiago/tiago_mujoco/model/tiago.urdf (robot description, URDF)
Before this commit: robot tiago, 89 links, 88 joints
Links:
- link arm_1_link: geometry collision mesh filename=package://tiago_description/meshes/arm/arm_1.stl scale=1 1 1; visual mesh filename=package://tiago_description/meshes/arm/arm_1_collision.dae scale=1 1 1
- link arm_2_link: geometry collision mesh filename=package://tiago_description/meshes/arm/arm_2.stl scale=1 1 1; visual mesh filename=package://tiago_description/meshes/arm/arm_2_collision.dae scale=1 1 1
- link arm_3_link: geometry collision mesh filename=package://tiago_description/meshes/arm/arm_3.stl scale=1 1 1; visual mesh filename=package://tiago_description/meshes/arm/arm_3_collision.dae scale=1 1 1
- link arm_4_link: geometry collision mesh filename=package://tiago_description/meshes/arm/arm_4.stl scale=1 1 1; visual mesh filename=package://tiago_description/meshes/arm/arm_4_collision.dae scale=1 1 1
- link arm_5_link: geometry collision mesh filename=package://tiago_description/meshes/arm/arm_5-wrist-2010.stl scale=1 1 1; visual mesh filename=package://tiago_description/meshes/arm/arm_5_collision-wris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 scale=1 1 1
- link arm_6_link: geometry collision mesh filename=package://tiago_description/meshes/arm/arm_6-wrist-2010.stl scale=1 1 1; visual mesh filename=package://tiago_description/meshes/arm/arm_6_collision-wris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 scale=1 1 1
- link head_1_link: geometry collision mesh filename=package://tiago_description/meshes/head/head_1.stl scale=1 1 1; visual mesh filename=package://tiago_description/meshes/head/head_1_collision.dae scale=1 1 1
- link head_2_link: geometry collision mesh filename=package://tiago_description/meshes/head/head_2.stl scale=1 1 1; visual mesh filename=package://tiago_description/meshes/head/head_2_collision.dae scale=1 1 1
- link torso_lift_link: geometry collision mesh filename=package://tiago_description/meshes/torso/torso_lift_with_ar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 scale=1 1 1; visual mesh filename=package://tiago_description/meshes/torso/torso_lift_collisi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 scale=1 1 1
