Commit message: Fix tiago

File: tiago/tiago_mujoco/model/tiago.urdf (robot description, URDF)
Before this commit: robot tiago, 89 links, 88 joints
Links:
- removed link arm_1_link
- removed link arm_2_link
- removed link arm_3_link
- removed link arm_4_link
- removed link arm_5_link
- removed link arm_6_link
- removed link arm_7_link
- removed link arm_tool_link
- removed link hand_grasping_frame
- removed link hand_index_abd_link
- removed link hand_index_flex_1_link
- removed link hand_index_flex_2_link
- removed link hand_index_flex_3_link
- removed link hand_index_link
- removed link hand_index_virtual_1_link
- removed link hand_index_virtual_2_link
- removed link hand_index_virtual_3_link
- removed link hand_little_abd_link
- removed link hand_little_flex_1_link
- removed link hand_little_flex_2_link
- removed link hand_little_flex_3_link
- removed link hand_little_virtual_1_link
- removed link hand_little_virtual_2_link
- removed link hand_little_virtual_3_link
- removed link hand_middle_abd_link
- removed link hand_middle_flex_1_link
- removed link hand_middle_flex_2_link
- removed link hand_middle_flex_3_link
- removed link hand_middle_virtual_1_link
- removed link hand_middle_virtual_2_link
- removed link hand_middle_virtual_3_link
- removed link hand_mrl_link
- removed link hand_palm_link
- removed link hand_ring_abd_link
- removed link hand_ring_flex_1_link
- removed link hand_ring_flex_2_link
- removed link hand_ring_flex_3_link
- removed link hand_ring_virtual_1_link
- removed link hand_ring_virtual_2_link
- removed link hand_ring_virtual_3_link
- removed link hand_safety_box
- removed link hand_thumb_abd_link
- removed link hand_thumb_flex_1_link
- removed link hand_thumb_flex_2_link
- removed link hand_thumb_link
- removed link hand_thumb_virtual_1_link
- removed link hand_thumb_virtual_2_link
- removed link hand_tool_link
- removed link wrist_ft_link
- removed link wrist_ft_tool_link
- added link arm_left_1_link, mass 1.563428; collision mesh filename=package://tiago_description/meshes/arm/arm_1_collision.dae scale=1 -1 -1; visual mesh filename=package://tiago_description/meshes/arm/arm_1.stl scale=1 -1 -1
- added link arm_left_2_link, mass 1.800397; collision mesh filename=package://tiago_description/meshes/arm/arm_2_collision.dae scale=1 1 -1; visual mesh filename=package://tiago_description/meshes/arm/arm_2.stl scale=1 1 -1
- added link arm_left_3_link, mass 1.8; collision mesh filename=package://tiago_description/meshes/arm/arm_3_collision.dae scale=1 1 -1; visual mesh filename=package://tiago_description/meshes/arm/arm_3.stl scale=1 1 -1
- added link arm_left_4_link, mass 1.432697; collision mesh filename=package://tiago_description/meshes/arm/arm_4_collision.dae scale=-1 -1 -1; visual mesh filename=package://tiago_description/meshes/arm/arm_4.stl scale=-1 -1 -1
- added link arm_left_5_link, mass 0.9359143689; collision mesh filename=package://tiago_description/meshes/arm/arm_5_collision-wris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 scale=-1 -1 -1; visual mesh filename=package://tiago_description/meshes/arm/arm_5-wrist-2017.stl scale=-1 -1 -1
- added link arm_left_6_link, mass 0.30275767222; collision mesh filename=package://tiago_description/meshes/arm/arm_6_collision-wris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 scale=-1 1 1; visual mesh filename=package://tiago_description/meshes/arm/arm_6-wrist-2017.stl scale=-1 1 1
- added link arm_left_7_link, mass 0.100
- added link arm_left_tool_link, mass 0.1; collision cylinder length=0.005 radius=0.005; visual cylinder length=0.005 radius=0.005
- added link arm_right_1_link, mass 1.563428; collision mesh filename=package://tiago_description/meshes/arm/arm_1_collision.dae scale=1 -1 1; visual mesh filename=package://tiago_description/meshes/arm/arm_1.stl scale=1 -1 1
- added link arm_right_2_link, mass 1.800397; collision mesh filename=package://tiago_description/meshes/arm/arm_2_collision.dae scale=1 1 1; visual mesh filename=package://tiago_description/meshes/arm/arm_2.stl scale=1 1 1
- added link arm_right_3_link, mass 1.8; collision mesh filename=package://tiago_description/meshes/arm/arm_3_collision.dae scale=1 1 1; visual mesh filename=package://tiago_description/meshes/arm/arm_3.stl scale=1 1 1
- added link arm_right_4_link, mass 1.432697; collision mesh filename=package://tiago_description/meshes/arm/arm_4_collision.dae scale=1 1 1; visual mesh filename=package://tiago_description/meshes/arm/arm_4.stl scale=1 1 1
- added link arm_right_5_link, mass 0.9359143689; collision mesh filename=package://tiago_description/meshes/arm/arm_5_collision-wris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 scale=1 1 1; visual mesh filename=package://tiago_description/meshes/arm/arm_5-wrist-2017.stl scale=1 1 1
- added link arm_right_6_link, mass 0.30275767222; collision mesh filename=package://tiago_description/meshes/arm/arm_6_collision-wris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 scale=1 1 1; visual mesh filename=package://tiago_description/meshes/arm/arm_6-wrist-2017.stl scale=1 1 1
- added link arm_right_7_link, mass 0.100
- added link arm_right_tool_link, mass 0.1; collision cylinder length=0.005 radius=0.005; visual cylinder length=0.005 radius=0.005
- added link gripper_left_grasping_frame, mass 0.0001
- added link gripper_left_left_finger_link, mass 0.109980; collision box size=0.01 0.05 0.11; visual mesh filename=package://pal_gripper_description/meshes/gripper_finger_lin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
- added link gripper_left_link, mass 0.602660; collision mesh filename=package://pal_gripper_description/meshes/gripper_link_colli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; visual mesh filename=package://pal_gripper_description/meshes/gripper_link.stl
- added link gripper_left_right_finger_link, mass 0.109980; collision box size=0.01 0.05 0.11; visual mesh filename=package://pal_gripper_description/meshes/gripper_finger_lin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 scale=-1 -1 1
- added link gripper_left_tool_link, mass 0.0001
- added link gripper_right_grasping_frame, mass 0.0001
- added link gripper_right_left_finger_link, mass 0.109980; collision box size=0.01 0.05 0.11; visual mesh filename=package://pal_gripper_description/meshes/gripper_finger_lin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
- added link gripper_right_link, mass 0.602660; collision mesh filename=package://pal_gripper_description/meshes/gripper_link_colli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; visual mesh filename=package://pal_gripper_description/meshes/gripper_link.stl
- added link gripper_right_right_finger_link, mass 0.109980; collision box size=0.01 0.05 0.11; visual mesh filename=package://pal_gripper_description/meshes/gripper_finger_lin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 scale=-1 -1 1
- added link gripper_right_tool_link, mass 0.0001
- added link wrist_left_ft_link, mass 0.1; collision cylinder length=0.0157 radius=0.0225; visual cylinder length=0.0157 radius=0.0225
- added link wrist_left_ft_tool_link, mass 0.1; collision cylinder length=0.00975 radius=0.025; visual cylinder length=0.00975 radius=0.025
- added link wrist_right_ft_link, mass 0.1; collision cylinder length=0.0157 radius=0.0225; visual cylinder length=0.0157 radius=0.0225
- added link wrist_right_ft_tool_link, mass 0.1; collision cylinder length=0.00975 radius=0.025; visual cylinder length=0.00975 radius=0.025
- link base_antenna_left_link: geometry collision cylinder length=0.17 radius=0.005; visual mesh filename=package://pmb2_description/meshes/objects/antenna.stl
- link base_antenna_right_link: geometry collision cylinder length=0.17 radius=0.005; visual mesh filename=package://pmb2_description/meshes/objects/antenna.stl
- link base_cover_link: geometry visual mesh filename=package://pmb2_description/meshes/base/base_ring.stl
- link base_laser_link: geometry visual mesh filename=package://pmb2_description/meshes/sensors/sick_tim551.stl
- link base_link: geometry collision mesh filename=package://pmb2_description/meshes/base/base_collision.stl; visual mesh filename=package://pmb2_description/meshes/base/base.stl
- link base_sonar_01_link: geometry visual mesh filename=package://pmb2_description/meshes/sensors/srf05.stl
- link base_sonar_02_link: geometry visual mesh filename=package://pmb2_description/meshes/sensors/srf05.stl
- link base_sonar_03_link: geometry visual mesh filename=package://pmb2_description/meshes/sensors/srf05.stl
- link caster_back_left_1_link: geometry visual mesh filename=package://pmb2_description/meshes/wheels/caster_1.stl
- link caster_back_left_2_link: geometry collision sphere radius=0.025; visual mesh filename=package://pmb2_description/meshes/wheels/caster_2.stl
- link caster_back_right_1_link: geometry visual mesh filename=package://pmb2_description/meshes/wheels/caster_1.stl
- link caster_back_right_2_link: geometry collision sphere radius=0.025; visual mesh filename=package://pmb2_description/meshes/wheels/caster_2.stl
- link caster_front_left_1_link: geometry visual mesh filename=package://pmb2_description/meshes/wheels/caster_1.stl
- link caster_front_left_2_link: geometry collision sphere radius=0.025; visual mesh filename=package://pmb2_description/meshes/wheels/caster_2.stl
- link caster_front_right_1_link: geometry visual mesh filename=package://pmb2_description/meshes/wheels/caster_1.stl
- link caster_front_right_2_link: geometry collision sphere radius=0.025; visual mesh filename=package://pmb2_description/meshes/wheels/caster_2.stl
- link head_1_link: geometry collision mesh filename=package://tiago_description/meshes/head/head_1_collision.dae scale=1 1 1; visual mesh filename=package://tiago_description/meshes/head/head_1.stl scale=1 1 1
- link head_2_link: geometry collision mesh filename=package://tiago_description/meshes/head/head_2_collision.dae scale=1 1 1; visual mesh filename=package://tiago_description/meshes/head/head_2.stl scale=1 1 1
- link torso_fixed_column_link: geometry collision box size=0.23 0.23 0.55; visual box size=0.18 0.2 0.55
- link torso_fixed_link: geometry collision box size=0.25 0.25 0.1; collision box size=0.4 0.25 0.04
- link torso_lift_link: mass 6.93198 -> 9.594213; geometry collision mesh filename=package://tiago_description/meshes/torso/torso_lift_collisi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 scale=1 1 1; collision mesh filename=package://tiago_description/meshes/torso/torso_lift_collisi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 scale=1 1 1
- link wheel_left_link: geometry collision sphere radius=0.0985; visual mesh filename=package://pmb2_description/meshes/wheels/wheel.stl
- link wheel_right_link: geometry collision sphere radius=0.0985; visual mesh filename=package://pmb2_description/meshes/wheels/wheel.stl
Joints:
- removed joint arm_1_joint
- removed joint arm_2_joint
- removed joint arm_3_joint
- removed joint arm_4_joint
- removed joint arm_5_joint
- removed joint arm_6_joint
- removed joint arm_7_joint
- removed joint arm_tool_joint
- removed joint hand_grasping_fixed_joint
- removed joint hand_index_abd_joint
- removed joint hand_index_flex_1_joint
- removed joint hand_index_flex_2_joint
- removed joint hand_index_flex_3_joint
- removed joint hand_index_joint
- removed joint hand_index_virtual_1_joint
- removed joint hand_index_virtual_2_joint
- removed joint hand_index_virtual_3_joint
- removed joint hand_little_abd_joint
- removed joint hand_little_flex_1_joint
- removed joint hand_little_flex_2_joint
- removed joint hand_little_flex_3_joint
- removed joint hand_little_virtual_1_joint
- removed joint hand_little_virtual_2_joint
- removed joint hand_little_virtual_3_joint
- removed joint hand_middle_abd_joint
- removed joint hand_middle_flex_1_joint
- removed joint hand_middle_flex_2_joint
- removed joint hand_middle_flex_3_joint
- removed joint hand_middle_virtual_1_joint
- removed joint hand_middle_virtual_2_joint
- removed joint hand_middle_virtual_3_joint
- removed joint hand_mrl_joint
- removed joint hand_palm_joint
- removed joint hand_ring_abd_joint
- removed joint hand_ring_flex_1_joint
- removed joint hand_ring_flex_2_joint
- removed joint hand_ring_flex_3_joint
- removed joint hand_ring_virtual_1_joint
- removed joint hand_ring_virtual_2_joint
- removed joint hand_ring_virtual_3_joint
- removed joint hand_safety_box_joint
- removed joint hand_thumb_abd_joint
- removed joint hand_thumb_flex_1_joint
- removed joint hand_thumb_flex_2_joint
- removed joint hand_thumb_joint
- removed joint hand_thumb_virtual_1_joint
- removed joint hand_thumb_virtual_2_joint
- removed joint hand_tool_joint
- removed joint wrist_ft_joint
- removed joint wrist_tool_joint
- added joint arm_left_1_joint: type revolute, parent torso_lift_link, child arm_left_1_link, origin xyz=0.02556 0.19 -0.171 rpy=3.141592653589793 0 1.5707963267948966, axis 0 0 1, limit lower=-1.1780972450961724 upper=1.5707963267948966 effort=43.0 velocity=1.95
- added joint arm_left_2_joint: type revolute, parent arm_left_1_link, child arm_left_2_link, origin xyz=0.125 -0.0195 0.031 rpy=1.5707963267948966 0.0 0.0, axis 0 0 1, limit lower=-1.1780972450961724 upper=1.5707963267948966 effort=43.0 velocity=1.95
- added joint arm_left_3_joint: type revolute, parent arm_left_2_link, child arm_left_3_link, origin xyz=0.0895 0.0 -0.0015 rpy=-1.5707963267948966 3.141592653589793 -1.5707963267948966, axis 0 0 1, limit lower=-0.7853981633974483 upper=3.9269908169872414 effort=26 velocity=2.35
- added joint arm_left_4_joint: type revolute, parent arm_left_3_link, child arm_left_4_link, origin xyz=-0.02 -0.027 0.222 rpy=1.5707963267948966 -1.5707963267948966 0.0, axis 0 0 1, limit lower=-0.39269908169872414 upper=2.356194490192345 effort=26 velocity=2.35
- added joint arm_left_5_joint: type revolute, parent arm_left_4_link, child arm_left_5_link, origin xyz=0.162 -0.02 -0.027 rpy=1.5707963267948966 -1.5707963267948966 -1.5707963267948966, axis 0 0 1, limit lower=-2.0943951023931953 upper=2.0943951023931953 effort=3 velocity=1.95
- added joint arm_left_6_joint: type revolute, parent arm_left_5_link, child arm_left_6_link, origin xyz=0 0 -0.15 rpy=0.0 -1.5707963267948966 -1.5707963267948966, axis 0 0 1, limit lower=-1.413716694115407 upper=1.413716694115407 effort=6.6 velocity=1.76
- added joint arm_left_7_joint: type revolute, parent arm_left_6_link, child arm_left_7_link, origin xyz=0 0 0 rpy=1.5707963267948966 0.0 1.5707963267948966, axis 0 0 1, limit lower=-2.0943951023931953 upper=2.0943951023931953 effort=6.6 velocity=1.76
- added joint arm_left_tool_joint: type fixed, parent arm_left_7_link, child arm_left_tool_link, origin xyz=0 0 -0.046 rpy=1.5707963267948966 1.5707963267948966 3.141592653589793
- added joint arm_right_1_joint: type revolute, parent torso_lift_link, child arm_right_1_link, origin xyz=0.02556 -0.19 -0.171 rpy=0 0 -1.5707963267948966, axis 0 0 1, limit lower=-1.1780972450961724 upper=1.5707963267948966 effort=43.0 velocity=1.95
- added joint arm_right_2_joint: type revolute, parent arm_right_1_link, child arm_right_2_link, origin xyz=0.125 -0.0195 -0.031 rpy=-1.5707963267948966 0.0 0.0, axis 0 0 1, limit lower=-1.1780972450961724 upper=1.5707963267948966 effort=43.0 velocity=1.95
- added joint arm_right_3_joint: type revolute, parent arm_right_2_link, child arm_right_3_link, origin xyz=0.0895 0.0 -0.0015 rpy=-1.5707963267948966 0.0 1.5707963267948966, axis 0 0 1, limit lower=-0.7853981633974483 upper=3.9269908169872414 effort=26 velocity=2.35
- added joint arm_right_4_joint: type revolute, parent arm_right_3_link, child arm_right_4_link, origin xyz=-0.02 -0.027 -0.222 rpy=-1.5707963267948966 -1.5707963267948966 0.0, axis 0 0 1, limit lower=-0.39269908169872414 upper=2.356194490192345 effort=26 velocity=2.35
- added joint arm_right_5_joint: type revolute, parent arm_right_4_link, child arm_right_5_link, origin xyz=-0.162 0.02 0.027 rpy=1.5707963267948966 -1.5707963267948966 -1.5707963267948966, axis 0 0 1, limit lower=-2.0943951023931953 upper=2.0943951023931953 effort=3 velocity=1.95
- added joint arm_right_6_joint: type revolute, parent arm_right_5_link, child arm_right_6_link, origin xyz=0 0 0.15 rpy=0.0 -1.5707963267948966 -1.5707963267948966, axis 0 0 1, limit lower=-1.413716694115407 upper=1.413716694115407 effort=6.6 velocity=1.76
- added joint arm_right_7_joint: type revolute, parent arm_right_6_link, child arm_right_7_link, origin xyz=0 0 0 rpy=1.5707963267948966 0.0 1.5707963267948966, axis 0 0 1, limit lower=-2.0943951023931953 upper=2.0943951023931953 effort=6.6 velocity=1.76
- added joint arm_right_tool_joint: type fixed, parent arm_right_7_link, child arm_right_tool_link, origin xyz=0 0 0.046 rpy=1.5707963267948966 -1.5707963267948966 3.141592653589793
- added joint gripper_left_grasping_frame_joint: type fixed, parent gripper_left_link, child gripper_left_grasping_frame, origin xyz=0 0 -0.12 rpy=-1.5708 1.5708 0
- added joint gripper_left_joint: type fixed, parent wrist_left_ft_tool_link, child gripper_left_link, origin xyz=0.01 0 0 rpy=1.5707963267948966 1.5707963267948966 -1.5707963267948966, axis 0 0 0
- added joint gripper_left_left_finger_joint: type prismatic, parent gripper_left_link, child gripper_left_left_finger_link, origin xyz=0. 0 0 rpy=0 0 0, axis -1 0 0, limit lower=0 upper=0.045 effort=16 velocity=0.05
- added joint gripper_left_right_finger_joint: type prismatic, parent gripper_left_link, child gripper_left_right_finger_link, origin xyz=0. 0 0 rpy=0 0 0, axis 1 0 0, limit lower=0.0 upper=0.045 effort=16 velocity=0.05
- added joint gripper_left_tool_joint: type fixed, parent wrist_left_ft_tool_link, child gripper_left_tool_link, origin xyz=0.01 0 0 rpy=1.5707963267948966 1.5707963267948966 -1.5707963267948966, axis 0 0 0
- added joint gripper_right_grasping_frame_joint: type fixed, parent gripper_right_link, child gripper_right_grasping_frame, origin xyz=0 0 -0.12 rpy=-1.5708 1.5708 0
- added joint gripper_right_joint: type fixed, parent wrist_right_ft_tool_link, child gripper_right_link, origin xyz=0.01 0 0 rpy=1.5707963267948966 1.5707963267948966 -1.5707963267948966, axis 0 0 0
- added joint gripper_right_left_finger_joint: type prismatic, parent gripper_right_link, child gripper_right_left_finger_link, origin xyz=0. 0 0 rpy=0 0 0, axis -1 0 0, limit lower=0 upper=0.045 effort=16 velocity=0.05
- added joint gripper_right_right_finger_joint: type prismatic, parent gripper_right_link, child gripper_right_right_finger_link, origin xyz=0. 0 0 rpy=0 0 0, axis 1 0 0, limit lower=0.0 upper=0.045 effort=16 velocity=0.05
- added joint gripper_right_tool_joint: type fixed, parent wrist_right_ft_tool_link, child gripper_right_tool_link, origin xyz=0.01 0 0 rpy=1.5707963267948966 1.5707963267948966 -1.5707963267948966, axis 0 0 0
- added joint wrist_left_ft_joint: type fixed, parent arm_left_tool_link, child wrist_left_ft_link, origin xyz=0.00785 0 0 rpy=1.5707963267948966 0 1.5707963267948966
- added joint wrist_left_tool_joint: type fixed, parent wrist_left_ft_link, child wrist_left_ft_tool_link, origin xyz=0 0 0.012725 rpy=-1.5707963267948966 -1.5707963267948966 0
- added joint wrist_right_ft_joint: type fixed, parent arm_right_tool_link, child wrist_right_ft_link, origin xyz=0.00785 0 0 rpy=1.5707963267948966 0 1.5707963267948966
- added joint wrist_right_tool_joint: type fixed, parent wrist_right_ft_link, child wrist_right_ft_tool_link, origin xyz=0 0 0.012725 rpy=-1.5707963267948966 -1.5707963267948966 0
