Commit message: Fix mir_system

File: mir_system/mir_system_description/mir100_hook_description/urdf/mir100_hook.urdf (robot description, URDF)
Before this commit: robot mir100_hook, 6 links, 5 joints
Joints:
- joint lift_arm_upper: axis 0 0 1.0 -> (none); limit lower=-1.5707964 upper=1.5707964 effort=100.0 velocity=6.0 -> (none); origin xyz=-0.0775113 0 0.0832461 rpy=1.5707964 0 0 -> xyz=-0.0775113 0 0.0832461 rpy=1.5707964 -0.26 0; type revolute -> fixed
- joint lift_motor_joint: axis 0 0 1.0 -> (none); limit lower=-0.5235988 upper=0.5235988 effort=100.0 velocity=6.0 -> (none); origin xyz=-0.1756014 0.1282467 3e-05 rpy=0 0 0 -> xyz=-0.1756014 0.1282467 3e-05 rpy=0 0 -0.13; type revolute -> fixed

File: mir_system/mir_system_description/mir_system_description/urdf/mir_system.urdf (robot description, URDF)
Before this commit: robot mir_system, 45 links, 44 joints
Joints:
- joint lift_arm_upper: axis 0 0 1.0 -> (none); limit lower=-1.5707964 upper=1.5707964 effort=100.0 velocity=6.0 -> (none); origin xyz=-0.0775113 0 0.0832461 rpy=1.5707964 0 0 -> xyz=-0.0775113 0 0.0832461 rpy=1.5707964 -0.26 0; type revolute -> fixed
- joint lift_motor_joint: axis 0 0 1.0 -> (none); limit lower=-0.5235988 upper=0.5235988 effort=100.0 velocity=6.0 -> (none); origin xyz=-0.1756014 0.1282467 3e-05 rpy=0 0 0 -> xyz=-0.1756014 0.1282467 3e-05 rpy=0 0 -0.13; type revolute -> fixed

Commit message: Add move_base

File: mir_system/mir_system_description/mir100_hook_description/urdf/mir100_hook.urdf (robot description, URDF)
Before this commit: robot mir100_hook, 6 links, 5 joints
Joints:
- joint carriage: limit lower=-0.5235988 upper=0 effort=0 velocity=0 -> lower=${-0.5235988+0.26} upper=0.26 effort=0 velocity=0; origin xyz=-0.418597 0.213663 3e-05 rpy=0 0 0 -> xyz=-0.418597 0.213663 3e-05 rpy=0 0 -0.26
- joint lift_arm_lower: limit lower=0 upper=0.5235988 effort=100.0 velocity=6.0 -> lower=-0.26 upper=${0.5235988-0.26} effort=100.0 velocity=6.0; origin xyz=-0.077511 3.3e-05 -0.0564022 rpy=1.5707964 0 0 -> xyz=-0.077511 3.3e-05 -0.0564022 rpy=1.5707964 -0.26 0

File: mir_system/mir_system_description/mir_description/urdf/mir.urdf (robot description, URDF)
Before this commit: robot mir_100, 22 links, 21 joints
Joints:
- joint base_link_to_back_laser_joint: origin xyz=-0.3548 -0.2352 0.1914 rpy=3.14159265359 0.0 -2.35619449019 -> xyz=-0.3548 -0.2352 0.1914 rpy=3.141592653589793 0.0 -2.356194490192345
- joint base_link_to_front_laser_joint: origin xyz=0.4288 0.2358 0.1914 rpy=3.14159265359 0.0 0.785398163397 -> xyz=0.4288 0.2358 0.1914 rpy=3.141592653589793 0.0 0.7853981633974483

File: mir_system/mir_system_description/mir_system_description/urdf/mir_system.urdf (robot description, URDF)
Before this commit: robot mir_system, 45 links, 44 joints
Joints:
- joint carriage: limit lower=-0.5235988 upper=0 effort=0 velocity=0 -> lower=-0.2635988 upper=0.26 effort=0 velocity=0; origin xyz=-0.418597 0.213663 3e-05 rpy=0 0 0 -> xyz=-0.418597 0.213663 3e-05 rpy=0 0 -0.26
- joint lift_arm_lower: limit lower=0 upper=0.5235988 effort=100.0 velocity=6.0 -> lower=-0.26 upper=0.2635988 effort=100.0 velocity=6.0; origin xyz=-0.077511 3.3e-05 -0.0564022 rpy=1.5707964 0 0 -> xyz=-0.077511 3.3e-05 -0.0564022 rpy=1.5707964 -0.26 0

Commit message: Fix mir_system and change use_odom_joints to add_odom_joints

File: mir_system/mir_system_description/mir100_hook_description/urdf/mir100_hook.urdf (robot description, URDF)
Before this commit: robot mir100_hook, 6 links, 5 joints
Joints:
- joint carriage: limit lower=${-0.5235988+0.26} upper=0.26 effort=0 velocity=0 -> lower=-0.5235988 upper=0 effort=0 velocity=0; origin xyz=-0.418597 0.213663 3e-05 rpy=0 0 -0.26 -> xyz=-0.418597 0.213663 3e-05 rpy=0 0 0
- joint lift_arm_lower: limit lower=-0.26 upper=${0.5235988-0.26} effort=100.0 velocity=6.0 -> lower=0 upper=0.5235988 effort=100.0 velocity=6.0; origin xyz=-0.077511 3.3e-05 -0.0564022 rpy=1.5707964 -0.26 0 -> xyz=-0.077511 3.3e-05 -0.0564022 rpy=1.5707964 0 0
- joint lift_arm_upper: axis (none) -> 0 0 1.0; limit (none) -> lower=-1.5707964 upper=1.5707964 effort=100.0 velocity=6.0; mimic (none) -> joint=lift_arm_lower multiplier=1.0; origin xyz=-0.0775113 0 0.0832461 rpy=1.5707964 -0.26 0 -> xyz=-0.0775113 0 0.0832461 rpy=1.5707964 0 0; type fixed -> revolute
- joint lift_motor_joint: axis (none) -> 0 0 1.0; limit (none) -> lower=-0.5235988 upper=0.5235988 effort=100.0 velocity=6.0; mimic (none) -> joint=lift_arm_lower multiplier=-0.5; origin xyz=-0.1756014 0.1282467 3e-05 rpy=0 0 -0.13 -> xyz=-0.1756014 0.1282467 3e-05 rpy=0 0 0; type fixed -> revolute

File: mir_system/mir_system_description/mir_system_description/urdf/mir_system.urdf (robot description, URDF)
Before this commit: robot mir_system, 45 links, 44 joints
Joints:
- joint carriage: limit lower=-0.2635988 upper=0.26 effort=0 velocity=0 -> lower=-0.5235988 upper=0 effort=0 velocity=0; origin xyz=-0.418597 0.213663 3e-05 rpy=0 0 -0.26 -> xyz=-0.418597 0.213663 3e-05 rpy=0 0 0
- joint lift_arm_lower: limit lower=-0.26 upper=0.2635988 effort=100.0 velocity=6.0 -> lower=0 upper=0.5235988 effort=100.0 velocity=6.0; origin xyz=-0.077511 3.3e-05 -0.0564022 rpy=1.5707964 -0.26 0 -> xyz=-0.077511 3.3e-05 -0.0564022 rpy=1.5707964 0 0
- joint lift_arm_upper: axis (none) -> 0 0 1.0; limit (none) -> lower=-1.5707964 upper=1.5707964 effort=100.0 velocity=6.0; mimic (none) -> joint=lift_arm_lower multiplier=1.0; origin xyz=-0.0775113 0 0.0832461 rpy=1.5707964 -0.26 0 -> xyz=-0.0775113 0 0.0832461 rpy=1.5707964 0 0; type fixed -> revolute
- joint lift_motor_joint: axis (none) -> 0 0 1.0; limit (none) -> lower=-0.5235988 upper=0.5235988 effort=100.0 velocity=6.0; mimic (none) -> joint=lift_arm_lower multiplier=-0.5; origin xyz=-0.1756014 0.1282467 3e-05 rpy=0 0 -0.13 -> xyz=-0.1756014 0.1282467 3e-05 rpy=0 0 0; type fixed -> revolute

Commit message: Fix bugs

File: mir_system/mir_system_description/mir100_hook_description/urdf/mir100_hook.urdf (robot description, URDF)
Before this commit: robot mir100_hook, 6 links, 5 joints
Joints:
- joint carriage: mimic (none) -> joint=lift_arm_lower multiplier=-1.0

File: mir_system/mir_system_description/mir_system_description/urdf/mir_system.urdf (robot description, URDF)
Before this commit: robot mir_system, 45 links, 44 joints
Joints:
- joint carriage: mimic (none) -> joint=lift_arm_lower multiplier=-1.0

File: mir_system/mir_system_mujoco/model/mir_system/meshes/mir_system.urdf (robot description, URDF)
Before this commit: robot mir_system, 45 links, 44 joints
Joints:
- joint carriage: mimic (none) -> joint=lift_arm_lower multiplier=-1.0
