Commit message: Add cartpole_control

File: cartpole/cartpole_mujoco/model/cartpole/meshes/cartpole.urdf (robot description, URDF)
Before this commit: robot physics, 5 links, 4 joints
Links:
- link pole: geometry collision cylinder length=1.0 radius=0.05; visual cylinder length=1.0 radius=0.05
Joints:
- joint cart_to_pole_x: limit lower=-6.28 upper=6.28 effort=100 velocity=3.14 -> (none); type revolute -> continuous
- joint pole_x_to_pole: limit lower=-6.28 upper=6.28 effort=100 velocity=3.14 -> (none); type revolute -> continuous

File: cartpole/cartpole_mujoco/urdf/cartpole.urdf (robot description, URDF)
Before this commit: robot physics, 5 links, 4 joints
Links:
- link pole: geometry collision cylinder length=1.0 radius=0.05; visual cylinder length=1.0 radius=0.05
Joints:
- joint cart_to_pole_x: limit lower=-6.28 upper=6.28 effort=100 velocity=3.14 -> (none); type revolute -> continuous
- joint pole_x_to_pole: limit lower=-6.28 upper=6.28 effort=100 velocity=3.14 -> (none); type revolute -> continuous
