Commit message: Update armar6

File: armar/armar_description/urdf/armar6_clean.urdf (robot description, URDF)
Before this commit: robot Armar6, 122 links, 121 joints
Links:
- added link LidarBack; visual mesh filename=package://armar_description/urdf/lidar.stl scale=1.00000 1.00000 1.00000
- added link LidarFront; visual mesh filename=package://armar_description/urdf/lidar.stl scale=1.00000 1.00000 1.00000
- link Platform: geometry collision mesh filename=package://armar_description/models/data/armar6_models/robot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 scale=1.00000 1.00000 1.00000; visual mesh filename=package://armar_description/urdf/platform_without_lidars.stl scale=1.00000 1.00000 1.00000
Joints:
- added joint LidarBackJoint: type fixed, parent Platform, child LidarBack, origin xyz=-0.300042 -0.450058 0.076964 rpy=0.0 0.0 3.1415
- added joint LidarFrontJoint: type fixed, parent Platform, child LidarFront, origin xyz=0.300042 0.450058 0.076964 rpy=0.0 0.0 0.0
- joint jointfix_67_4: origin xyz=0.00000 0.00000 0.00000 rpy=0.00000 -0.00000 0.00000 -> xyz=0.00000 0.00000 0.00000 rpy=0.00000 -0.00000 -1.5707963267948966

Commit message: update armar

File: armar/armar_description/urdf/armar6_clean.urdf (robot description, URDF)
Before this commit: robot armar6, 124 links, 123 joints
Links:
- removed link Index L 1 Joint~Index L 1 Body
- removed link Index L 2 Joint~Index L 2 Body
- removed link Index L 3 Joint~Index L 3 Body
- removed link Index R 1 Joint~Index R 1 Body
- removed link Index R 2 Joint~Index R 2 Body
- removed link Index R 3 Joint~Index R 3 Body
- removed link Middle L 1 Joint~Middle L 1 Body
- removed link Middle L 2 Joint~Middle L 2 Body
- removed link Middle L 3 Joint~Middle L 3 Body
- removed link Middle R 1 Joint~Middle R 1 Body
- removed link Middle R 2 Joint~Middle R 2 Body
- removed link Middle R 3 Joint~Middle R 3 Body
- removed link Pinky L 1 Joint~Pinky L 1 Body
- removed link Pinky L 2 Joint~Pinky L 2 Body
- removed link Pinky L 3 Joint~Pinky L 3 Body
- removed link Pinky R 1 Joint~Pinky R 1 Body
- removed link Pinky R 2 Joint~Pinky R 2 Body
- removed link Pinky R 3 Joint~Pinky R 3 Body
- removed link Ring L 1 Joint~Ring L 1 Body
- removed link Ring L 2 Joint~Ring L 2 Body
- removed link Ring L 3 Joint~Ring L 3 Body
- removed link Ring R 1 Joint~Ring R 1 Body
- removed link Ring R 2 Joint~Ring R 2 Body
- removed link Ring R 3 Joint~Ring R 3 Body
- removed link Thumb L 1 Joint~Thumb L 1 Body
- removed link Thumb L 2 Joint~Thumb L 2 Body
- removed link Thumb R 1 Joint~Thumb R 1 Body
- removed link Thumb R 2 Joint~Thumb R 2 Body
- added link Index_L_1_Joint~Index L 1 Body; collision mesh filename=package://armar_description/models/data/armar6_models/robot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 scale=1.00000 1.00000 1.00000; visual mesh filename=package://armar_description/models/data/armar6_models/robot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 scale=1.00000 1.00000 1.00000
- added link Index_L_2_Joint~Index L 2 Body; collision mesh filename=package://armar_description/models/data/armar6_models/robot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 scale=1.00000 1.00000 1.00000; visual mesh filename=package://armar_description/models/data/armar6_models/robot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 scale=1.00000 1.00000 1.00000
- added link Index_L_3_Joint~Index L 3 Body; collision mesh filename=package://armar_description/models/data/armar6_models/robot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 scale=1.00000 1.00000 1.00000; visual mesh filename=package://armar_description/models/data/armar6_models/robot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 scale=1.00000 1.00000 1.00000
- added link Index_R_1_Joint~Index R 1 Body; collision mesh filename=package://armar_description/models/data/armar6_models/robot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 scale=1.00000 1.00000 1.00000; visual mesh filename=package://armar_description/models/data/armar6_models/robot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 scale=1.00000 1.00000 1.00000
- added link Index_R_2_Joint~Index R 2 Body; collision mesh filename=package://armar_description/models/data/armar6_models/robot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 scale=1.00000 1.00000 1.00000; visual mesh filename=package://armar_description/models/data/armar6_models/robot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 scale=1.00000 1.00000 1.00000
- added link Index_R_3_Joint~Index R 3 Body; collision mesh filename=package://armar_description/models/data/armar6_models/robot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 scale=1.00000 1.00000 1.00000; visual mesh filename=package://armar_description/models/data/armar6_models/robot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 scale=1.00000 1.00000 1.00000
- added link Middle_L_1_Joint~Middle L 1 Body; collision mesh filename=package://armar_description/models/data/armar6_models/robot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 scale=1.00000 1.00000 1.00000; visual mesh filename=package://armar_description/models/data/armar6_models/robot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 scale=1.00000 1.00000 1.00000
- added link Middle_L_2_Joint~Middle L 2 Body; collision mesh filename=package://armar_description/models/data/armar6_models/robot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 scale=1.00000 1.00000 1.00000; visual mesh filename=package://armar_description/models/data/armar6_models/robot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 scale=1.00000 1.00000 1.00000
- added link Middle_L_3_Joint~Middle L 3 Body; collision mesh filename=package://armar_description/models/data/armar6_models/robot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 scale=1.00000 1.00000 1.00000; visual mesh filename=package://armar_description/models/data/armar6_models/robot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 scale=1.00000 1.00000 1.00000
- added link Middle_R_1_Joint~Middle R 1 Body; collision mesh filename=package://armar_description/models/data/armar6_models/robot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 scale=1.00000 1.00000 1.00000; visual mesh filename=package://armar_description/models/data/armar6_models/robot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 scale=1.00000 1.00000 1.00000
- added link Middle_R_2_Joint~Middle R 2 Body; collision mesh filename=package://armar_description/models/data/armar6_models/robot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 scale=1.00000 1.00000 1.00000; visual mesh filename=package://armar_description/models/data/armar6_models/robot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 scale=1.00000 1.00000 1.00000
- added link Middle_R_3_Joint~Middle R 3 Body; collision mesh filename=package://armar_description/models/data/armar6_models/robot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 scale=1.00000 1.00000 1.00000; visual mesh filename=package://armar_description/models/data/armar6_models/robot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 scale=1.00000 1.00000 1.00000
- added link Pinky_L_1_Joint~Pinky L 1 Body; collision mesh filename=package://armar_description/models/data/armar6_models/robot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 scale=1.00000 1.00000 1.00000; visual mesh filename=package://armar_description/models/data/armar6_models/robot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 scale=1.00000 1.00000 1.00000
- added link Pinky_L_2_Joint~Pinky L 2 Body; collision mesh filename=package://armar_description/models/data/armar6_models/robot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 scale=1.00000 1.00000 1.00000; visual mesh filename=package://armar_description/models/data/armar6_models/robot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 scale=1.00000 1.00000 1.00000
- added link Pinky_L_3_Joint~Pinky L 3 Body; collision mesh filename=package://armar_description/models/data/armar6_models/robot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 scale=1.00000 1.00000 1.00000; visual mesh filename=package://armar_description/models/data/armar6_models/robot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 scale=1.00000 1.00000 1.00000
- added link Pinky_R_1_Joint~Pinky R 1 Body; collision mesh filename=package://armar_description/models/data/armar6_models/robot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 scale=1.00000 1.00000 1.00000; visual mesh filename=package://armar_description/models/data/armar6_models/robot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 scale=1.00000 1.00000 1.00000
- added link Pinky_R_2_Joint~Pinky R 2 Body; collision mesh filename=package://armar_description/models/data/armar6_models/robot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 scale=1.00000 1.00000 1.00000; visual mesh filename=package://armar_description/models/data/armar6_models/robot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 scale=1.00000 1.00000 1.00000
- added link Pinky_R_3_Joint~Pinky R 3 Body; collision mesh filename=package://armar_description/models/data/armar6_models/robot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 scale=1.00000 1.00000 1.00000; visual mesh filename=package://armar_description/models/data/armar6_models/robot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 scale=1.00000 1.00000 1.00000
- added link Ring_L_1_Joint~Ring L 1 Body; collision mesh filename=package://armar_description/models/data/armar6_models/robot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 scale=1.00000 1.00000 1.00000; visual mesh filename=package://armar_description/models/data/armar6_models/robot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 scale=1.00000 1.00000 1.00000
- added link Ring_L_2_Joint~Ring L 2 Body; collision mesh filename=package://armar_description/models/data/armar6_models/robot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 scale=1.00000 1.00000 1.00000; visual mesh filename=package://armar_description/models/data/armar6_models/robot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 scale=1.00000 1.00000 1.00000
- added link Ring_L_3_Joint~Ring L 3 Body; collision mesh filename=package://armar_description/models/data/armar6_models/robot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 scale=1.00000 1.00000 1.00000; visual mesh filename=package://armar_description/models/data/armar6_models/robot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 scale=1.00000 1.00000 1.00000
- added link Ring_R_1_Joint~Ring R 1 Body; collision mesh filename=package://armar_description/models/data/armar6_models/robot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 scale=1.00000 1.00000 1.00000; visual mesh filename=package://armar_description/models/data/armar6_models/robot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 scale=1.00000 1.00000 1.00000
- added link Ring_R_2_Joint~Ring R 2 Body; collision mesh filename=package://armar_description/models/data/armar6_models/robot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 scale=1.00000 1.00000 1.00000; visual mesh filename=package://armar_description/models/data/armar6_models/robot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 scale=1.00000 1.00000 1.00000
- added link Ring_R_3_Joint~Ring R 3 Body; collision mesh filename=package://armar_description/models/data/armar6_models/robot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 scale=1.00000 1.00000 1.00000; visual mesh filename=package://armar_description/models/data/armar6_models/robot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 scale=1.00000 1.00000 1.00000
- added link Thumb_L_1_Joint~Thumb L 1 Body; collision mesh filename=package://armar_description/models/data/armar6_models/robot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 scale=1.00000 1.00000 1.00000; visual mesh filename=package://armar_description/models/data/armar6_models/robot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 scale=1.00000 1.00000 1.00000
- added link Thumb_L_2_Joint~Thumb L 2 Body; collision mesh filename=package://armar_description/models/data/armar6_models/robot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 scale=1.00000 1.00000 1.00000; visual mesh filename=package://armar_description/models/data/armar6_models/robot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 scale=1.00000 1.00000 1.00000
- added link Thumb_R_1_Joint~Thumb R 1 Body; collision mesh filename=package://armar_description/models/data/armar6_models/robot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 scale=1.00000 1.00000 1.00000; visual mesh filename=package://armar_description/models/data/armar6_models/robot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 scale=1.00000 1.00000 1.00000
- added link Thumb_R_2_Joint~Thumb R 2 Body; collision mesh filename=package://armar_description/models/data/armar6_models/robot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 scale=1.00000 1.00000 1.00000; visual mesh filename=package://armar_description/models/data/armar6_models/robot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 scale=1.00000 1.00000 1.00000
Joints:
- removed joint Index L 1 Joint
- removed joint Index L 2 Joint
- removed joint Index L 3 Joint
- removed joint Index R 1 Joint
- removed joint Index R 2 Joint
- removed joint Index R 3 Joint
- removed joint Middle L 1 Joint
- removed joint Middle L 2 Joint
- removed joint Middle L 3 Joint
- removed joint Middle R 1 Joint
- removed joint Middle R 2 Joint
- removed joint Middle R 3 Joint
- removed joint Pinky L 1 Joint
- removed joint Pinky L 2 Joint
- removed joint Pinky L 3 Joint
- removed joint Pinky R 1 Joint
- removed joint Pinky R 2 Joint
- removed joint Pinky R 3 Joint
- removed joint Ring L 1 Joint
- removed joint Ring L 2 Joint
- removed joint Ring L 3 Joint
- removed joint Ring R 1 Joint
- removed joint Ring R 2 Joint
- removed joint Ring R 3 Joint
- removed joint Thumb L 1 Joint
- removed joint Thumb L 2 Joint
- removed joint Thumb R 1 Joint
- removed joint Thumb R 2 Joint
- added joint Index_L_1_Joint: type continuous, parent Hand L Palm, child link0_30, origin xyz=0.14531 -0.00000 0.03922 rpy=-1.57081 1.48348 -0.00001, axis 1.00000 0.00000 0.00000
- added joint Index_L_2_Joint: type continuous, parent Index_L_1_Joint~Index L 1 Body, child link0_32, origin xyz=0.00000 -0.05595 -0.00000 rpy=0.00000 -0.00000 0.00000, axis 1.00000 0.00000 0.00000
- added joint Index_L_3_Joint: type continuous, parent Index_L_2_Joint~Index L 2 Body, child link0_34, origin xyz=0.00000 -0.03197 -0.00000 rpy=0.00000 -0.00000 0.00000, axis 1.00000 0.00000 0.00000
- added joint Index_R_1_Joint: type continuous, parent Hand R Palm, child link0_82, origin xyz=0.14531 0.00000 -0.03922 rpy=1.57081 1.48348 -3.14158, axis 1.00000 0.00000 0.00000
- added joint Index_R_2_Joint: type continuous, parent Index_R_1_Joint~Index R 1 Body, child link0_84, origin xyz=0.00000 -0.05595 -0.00000 rpy=0.00000 -0.00000 0.00000, axis 1.00000 0.00000 0.00000
- added joint Index_R_3_Joint: type continuous, parent Index_R_2_Joint~Index R 2 Body, child link0_86, origin xyz=0.00000 -0.03197 -0.00000 rpy=0.00000 -0.00000 0.00000, axis 1.00000 0.00000 0.00000
- added joint Middle_L_1_Joint: type continuous, parent Hand L Palm, child link0_40, origin xyz=0.15172 0.00000 0.00750 rpy=0.00000 1.57080 -4.71239, axis 1.00000 0.00000 0.00000
- added joint Middle_L_2_Joint: type continuous, parent Middle_L_1_Joint~Middle L 1 Body, child link0_42, origin xyz=0.00000 -0.06000 0.00000 rpy=0.00000 -0.00000 0.00000, axis 1.00000 0.00000 0.00000
- added joint Middle_L_3_Joint: type continuous, parent Middle_L_2_Joint~Middle L 2 Body, child link0_44, origin xyz=0.00000 -0.03900 0.00000 rpy=0.00000 -0.00000 0.00000, axis 1.00000 0.00000 0.00000
- added joint Middle_R_1_Joint: type continuous, parent Hand R Palm, child link0_88, origin xyz=0.15172 0.00000 -0.00750 rpy=0.00000 1.57080 -4.71239, axis 1.00000 0.00000 0.00000
- added joint Middle_R_2_Joint: type continuous, parent Middle_R_1_Joint~Middle R 1 Body, child link0_90, origin xyz=0.00000 -0.06000 0.00000 rpy=0.00000 -0.00000 0.00000, axis 1.00000 0.00000 0.00000
- added joint Middle_R_3_Joint: type continuous, parent Middle_R_2_Joint~Middle R 2 Body, child link0_92, origin xyz=0.00000 -0.03900 0.00000 rpy=0.00000 -0.00000 0.00000, axis 1.00000 0.00000 0.00000
- added joint Pinky_L_1_Joint: type continuous, parent Hand L Palm, child link0_46, origin xyz=0.13032 -0.00000 -0.05530 rpy=1.57080 1.16969 3.14159, axis 1.00000 0.00000 0.00000
- added joint Pinky_L_2_Joint: type continuous, parent Pinky_L_1_Joint~Pinky L 1 Body, child link0_48, origin xyz=-0.00000 -0.04610 0.00000 rpy=0.00000 -0.00000 0.00000, axis 1.00000 0.00000 0.00000
- added joint Pinky_L_3_Joint: type continuous, parent Pinky_L_2_Joint~Pinky L 2 Body, child link0_50, origin xyz=-0.00000 -0.02706 0.00000 rpy=0.00000 -0.00000 0.00000, axis 1.00000 0.00000 0.00000
- added joint Pinky_R_1_Joint: type continuous, parent Hand R Palm, child link0_94, origin xyz=0.13032 0.00000 0.05530 rpy=-1.57080 1.16969 0.00000, axis 1.00000 0.00000 0.00000
- added joint Pinky_R_2_Joint: type continuous, parent Pinky_R_1_Joint~Pinky R 1 Body, child link0_96, origin xyz=0.00000 -0.04610 0.00000 rpy=0.00000 -0.00000 0.00000, axis 1.00000 0.00000 0.00000
- added joint Pinky_R_3_Joint: type continuous, parent Pinky_R_2_Joint~Pinky R 2 Body, child link0_98, origin xyz=0.00000 -0.02706 -0.00000 rpy=0.00000 -0.00000 0.00000, axis 1.00000 0.00000 0.00000
- added joint Ring_L_1_Joint: type continuous, parent Hand L Palm, child link0_52, origin xyz=0.14652 0.00000 -0.02630 rpy=1.57080 1.39616 3.14159, axis 1.00000 0.00000 0.00000
- added joint Ring_L_2_Joint: type continuous, parent Ring_L_1_Joint~Ring L 1 Body, child link0_54, origin xyz=0.00000 -0.05506 0.00000 rpy=0.00000 -0.00000 0.00000, axis 1.00000 0.00000 0.00000
- added joint Ring_L_3_Joint: type continuous, parent Ring_L_2_Joint~Ring L 2 Body, child link0_56, origin xyz=0.00000 -0.03704 0.00000 rpy=0.00000 -0.00000 0.00000, axis 1.00000 0.00000 0.00000
- added joint Ring_R_1_Joint: type continuous, parent Hand R Palm, child link0_104, origin xyz=0.14652 0.00000 0.02630 rpy=-1.57080 1.39616 0.00000, axis 1.00000 0.00000 0.00000
- added joint Ring_R_2_Joint: type continuous, parent Ring_R_1_Joint~Ring R 1 Body, child link0_106, origin xyz=0.00000 -0.05506 0.00000 rpy=0.00000 -0.00000 0.00000, axis 1.00000 0.00000 0.00000
- added joint Ring_R_3_Joint: type continuous, parent Ring_R_2_Joint~Ring R 2 Body, child link0_108, origin xyz=-0.00000 -0.03704 0.00000 rpy=0.00000 -0.00000 0.00000, axis 1.00000 0.00000 0.00000
- added joint Thumb_L_1_Joint: type continuous, parent Hand L Palm, child link0_58, origin xyz=0.08111 -0.04691 0.03950 rpy=-0.22370 -1.18631 0.20756, axis 1.00000 0.00000 0.00000
- added joint Thumb_L_2_Joint: type continuous, parent Thumb_L_1_Joint~Thumb L 1 Body, child link0_60, origin xyz=0.00002 -0.04408 -0.00005 rpy=0.00000 -0.00000 0.00000, axis 1.00000 0.00000 0.00000
- added joint Thumb_R_1_Joint: type continuous, parent Hand R Palm, child link0_110, origin xyz=0.08111 -0.04691 -0.03950 rpy=2.91903 -1.18743 -2.93505, axis 1.00000 0.00000 0.00000
- added joint Thumb_R_2_Joint: type continuous, parent Thumb_R_1_Joint~Thumb R 1 Body, child link0_112, origin xyz=-0.00002 -0.04408 -0.00005 rpy=0.00000 -0.00000 0.00000, axis 1.00000 0.00000 0.00000
- joint jointfix_10_48: child Pinky L 2 Joint~Pinky L 2 Body -> Pinky_L_2_Joint~Pinky L 2 Body
- joint jointfix_11_46: child Pinky L 1 Joint~Pinky L 1 Body -> Pinky_L_1_Joint~Pinky L 1 Body
- joint jointfix_12_56: child Ring L 3 Joint~Ring L 3 Body -> Ring_L_3_Joint~Ring L 3 Body
- joint jointfix_13_54: child Ring L 2 Joint~Ring L 2 Body -> Ring_L_2_Joint~Ring L 2 Body
- joint jointfix_14_52: child Ring L 1 Joint~Ring L 1 Body -> Ring_L_1_Joint~Ring L 1 Body
- joint jointfix_15_60: child Thumb L 2 Joint~Thumb L 2 Body -> Thumb_L_2_Joint~Thumb L 2 Body
- joint jointfix_16_58: child Thumb L 1 Joint~Thumb L 1 Body -> Thumb_L_1_Joint~Thumb L 1 Body
- joint jointfix_1_34: child Index L 3 Joint~Index L 3 Body -> Index_L_3_Joint~Index L 3 Body
- joint jointfix_29_86: child Index R 3 Joint~Index R 3 Body -> Index_R_3_Joint~Index R 3 Body
- joint jointfix_2_32: child Index L 2 Joint~Index L 2 Body -> Index_L_2_Joint~Index L 2 Body
- joint jointfix_30_84: child Index R 2 Joint~Index R 2 Body -> Index_R_2_Joint~Index R 2 Body
- joint jointfix_31_82: child Index R 1 Joint~Index R 1 Body -> Index_R_1_Joint~Index R 1 Body
- joint jointfix_32_92: child Middle R 3 Joint~Middle R 3 Body -> Middle_R_3_Joint~Middle R 3 Body
- joint jointfix_33_90: child Middle R 2 Joint~Middle R 2 Body -> Middle_R_2_Joint~Middle R 2 Body
- joint jointfix_34_88: child Middle R 1 Joint~Middle R 1 Body -> Middle_R_1_Joint~Middle R 1 Body
- joint jointfix_35_98: child Pinky R 3 Joint~Pinky R 3 Body -> Pinky_R_3_Joint~Pinky R 3 Body
- joint jointfix_36_96: child Pinky R 2 Joint~Pinky R 2 Body -> Pinky_R_2_Joint~Pinky R 2 Body
- joint jointfix_37_94: child Pinky R 1 Joint~Pinky R 1 Body -> Pinky_R_1_Joint~Pinky R 1 Body
- joint jointfix_3_30: child Index L 1 Joint~Index L 1 Body -> Index_L_1_Joint~Index L 1 Body
- joint jointfix_40_108: child Ring R 3 Joint~Ring R 3 Body -> Ring_R_3_Joint~Ring R 3 Body
- joint jointfix_41_106: child Ring R 2 Joint~Ring R 2 Body -> Ring_R_2_Joint~Ring R 2 Body
- joint jointfix_42_104: child Ring R 1 Joint~Ring R 1 Body -> Ring_R_1_Joint~Ring R 1 Body
- joint jointfix_43_112: child Thumb R 2 Joint~Thumb R 2 Body -> Thumb_R_2_Joint~Thumb R 2 Body
- joint jointfix_44_110: child Thumb R 1 Joint~Thumb R 1 Body -> Thumb_R_1_Joint~Thumb R 1 Body
- joint jointfix_6_44: child Middle L 3 Joint~Middle L 3 Body -> Middle_L_3_Joint~Middle L 3 Body
- joint jointfix_7_42: child Middle L 2 Joint~Middle L 2 Body -> Middle_L_2_Joint~Middle L 2 Body
- joint jointfix_8_40: child Middle L 1 Joint~Middle L 1 Body -> Middle_L_1_Joint~Middle L 1 Body
- joint jointfix_9_50: child Pinky L 3 Joint~Pinky L 3 Body -> Pinky_L_3_Joint~Pinky L 3 Body
